Commit message: Add files via upload

File: UCV_robot_urdf_description/urdf/UCV_robot_urdf.xacro (robot description, xacro)
@@ -6,7 +6,7 @@
 <link name="base_link">
   <inertial>
-    <origin xyz="-0.0028423334837031655 8.430721147465176e-06 0.004434783297020629" rpy="0 0 0"/>
-    <mass value="0.3635670282557214"/>
-    <inertia ixx="0.000485" iyy="0.000123" izz="0.000603" ixy="0.0" iyz="0.0" ixz="0.0"/>
+    <origin xyz="0.0005684663800967518 1.6861442325029684e-06 0.00477855003731065" rpy="0 0 0"/>
+    <mass value="5.453505423835813"/>
+    <inertia ixx="0.066842" iyy="0.046567" izz="0.113336" ixy="-0.0" iyz="-0.0" ixz="8.3e-05"/>
   </inertial>
   <visual>
@@ -24,3 +24,28 @@
   </collision>
 </link>
+<link name="Thigh_Ball_Bearing_v3_1">
+  <inertial>
+    <origin xyz="0.020631339541226576 -0.00715732305135211 0.0022868632249262114" rpy="0 0 0"/>
+    <mass value="0.06928040709442683"/>
+    <inertia ixx="1.6e-05" iyy="1.4e-05" izz="3e-05" ixy="9e-06" iyz="-0.0" ixz="0.0"/>
+  </inertial>
+  <visual>
+    <origin xyz="-0.035 0.164 -0.009" rpy="0 0 0"/>
+    <geometry>
+      <mesh filename="package://UCV_robot_urdf_description/meshes/Thigh_Ball_Bearing_v3_1.stl" scale="0.001 0.001 0.001"/>
+    </geometry>
+    <material name="silver"/>
+  </visual>
+  <collision>
+    <origin xyz="-0.035 0.164 -0.009" rpy="0 0 0"/>
+    <geometry>
+      <mesh filename="package://UCV_robot_urdf_description/meshes/Thigh_Ball_Bearing_v3_1.stl" scale="0.001 0.001 0.001"/>
+    </geometry>
+  </collision>
+</link>
+<joint name="Rigid 1" type="fixed">
+  <origin xyz="0.035 -0.164 0.009" rpy="0 0 0"/>
+  <parent link="base_link"/>
+  <child link="Thigh_Ball_Bearing_v3_1"/>
+</joint>
 </robot>
